Commit message: LAUNCH FILE WORKING

File: HMS_Perception/src/description/HMS_Perception_description.urdf (robot description, URDF)
Before this commit: robot rover, 3 links, 2 joints
Links:
- removed link body
- removed link imu_link
- added link base_footprint
- added link camera, mass 1; collision box size=0.1914947774659249 0.6346109922118176 0.19215263167384591; visual box size=0.1914947774659249 0.6346109922118176 0.19215263167384591
- added link imu_sensor, mass 1; collision box size=0.46603382719539876 0.45619487184483365 0.3454197767248413; visual box size=0.46603382719539876 0.45619487184483365 0.3454197767248413
- added link lidar, mass 1; collision cylinder length=0.13538975482266932 radius=0.333099402958804; visual cylinder length=0.13538975482266932 radius=0.333099402958804
- added link wheel_0, mass 1; collision cylinder length=0.05383527298985801 radius=0.2879384563584746; visual cylinder length=0.05383527298985801 radius=0.2879384563584746
- added link wheel_1, mass 1; collision cylinder length=0.05383527298985801 radius=0.2879384563584746; visual cylinder length=0.05383527298985801 radius=0.2879384563584746
- added link wheel_2, mass 1; collision cylinder length=0.05383527298985801 radius=0.2879384563584746; visual cylinder length=0.05383527298985801 radius=0.2879384563584746
- added link wheel_3, mass 1; collision cylinder length=0.05383527298985801 radius=0.2879384563584746; visual cylinder length=0.05383527298985801 radius=0.2879384563584746
- added link wheel_4, mass 1; collision cylinder length=0.05383527298985801 radius=0.2879384563584746; visual cylinder length=0.05383527298985801 radius=0.2879384563584746
- added link wheel_5, mass 1; collision cylinder length=0.05383527298985801 radius=0.2879384563584746; visual cylinder length=0.05383527298985801 radius=0.2879384563584746
- link base_link: mass None -> 1; geometry collision box size=3.7939062066566853 2.2800234239081933 0.5232328098292442; visual box size=3.794 2.28 0.523
Joints:
- removed joint base_link_to_chasis
- removed joint imu_joint
- added joint base_joint: type fixed, parent base_footprint, child base_link, origin xyz=0.000047751989472821776 0 1.5 rpy=0 0 0
- added joint base_link_to_camera: type fixed, parent base_link, child camera, origin xyz=1.6256258584357346 -0.02298885073006307 0.3695319117946291 rpy=0 0 0
- added joint base_link_to_imu_sensor: type fixed, parent base_link, child imu_sensor, origin xyz=-1.1282184172017464 0.06064584319013511 0.17904669409114127 rpy=0 0 0
- added joint base_link_to_lidar: type fixed, parent base_link, child lidar, origin xyz=0 0 0.2569669071788341 rpy=0 0 0
- added joint base_link_to_wheel_0: type continuous, parent base_link, child wheel_0, origin xyz=1.39 1.1909017501403918 -1 rpy=1.5707963267948963 0 0, axis 0 0 1
- added joint base_link_to_wheel_1: type continuous, parent base_link, child wheel_1, origin xyz=1.39 -1.17 -1 rpy=1.5707963267948963 0 0, axis 0 0 1
- added joint base_link_to_wheel_2: type continuous, parent base_link, child wheel_2, origin xyz=0 1.1909017501403918 -1 rpy=1.5707963267948963 0 0, axis 0 0 1
- added joint base_link_to_wheel_3: type continuous, parent base_link, child wheel_3, origin xyz=0.0005487795717144736 -1.1705640351243605 -1 rpy=1.5707963267948963 0 0, axis 0 0 1
- added joint base_link_to_wheel_4: type continuous, parent base_link, child wheel_4, origin xyz=-1.39 1.1909017501403918 -1 rpy=1.5707963267948963 0 0, axis 0 0 1
- added joint base_link_to_wheel_5: type continuous, parent base_link, child wheel_5, origin xyz=-1.39 -1.1736814480844906 -1 rpy=1.5707963267948963 0 0, axis 0 0 1
