Commit message: yolo

File: arm_assembly/src/description/arm_assembly.urdf (robot description, URDF)
Before this commit: robot arm_assembly, 352 links, 352 joints
Links:
- removed link 15mm_shaft
- removed link 17hs15_1504s1
- removed link 17hs15_1504s1_1
- removed link 1zgj4
- removed link 1zgj4_1
- removed link 1zgj4_10
- removed link 1zgj4_11
- removed link 1zgj4_2
- removed link 1zgj4_3
- removed link 1zgj4_4
- removed link 1zgj4_5
- removed link 1zgj4_6
- removed link 1zgj4_7
- removed link 1zgj4_8
- removed link 1zgj4_9
- removed link 2600n2_metal_miter_gear
- removed link 2600n2_metal_miter_gear_1
- removed link 2600n2_metal_miter_gear_2
- removed link 7769n12_timing_belt_idler_pulley
- removed link 7769n12_timing_belt_idler_pulley_1
- removed link 92010a328_passivated_18_8_stainless_steel_phillips_flat_head_screw_11
- removed link 92010a328_passivated_18_8_stainless_steel_phillips_flat_head_screw_12
- removed link 92010a328_passivated_18_8_stainless_steel_phillips_flat_head_screw_13
- removed link 92010a328_passivated_18_8_stainless_steel_phillips_flat_head_screw_14
- removed link 92010a328_passivated_18_8_stainless_steel_phillips_flat_head_screw_18
- removed link 92010a328_passivated_18_8_stainless_steel_phillips_flat_head_screw_3
- removed link 92010a328_passivated_18_8_stainless_steel_phillips_flat_head_screw_4
- removed link 92010a328_passivated_18_8_stainless_steel_phillips_flat_head_screw_7
- removed link 92010a328_passivated_18_8_stainless_steel_phillips_flat_head_screw_9
- removed link afbd19_30w_wb
- removed link afbd19_30w_wb_1
- removed link arm
- removed link arm_base_belt
- removed link atp18xl050_a_puf_a
- removed link atp18xl050_a_puf_a_1
- removed link atp60xl050_a_puh_a
- removed link atp72xl050_a_puh_a
- removed link bearing
- removed link bearing_2
- removed link bearing_3
- removed link bearing_688
- removed link bearing_688_1
- removed link bearing_688_1_1
- removed link body
- removed link body_1
- removed link body_2
- removed link button
- removed link cylindrical_10_0
- removed link cylindrical_12_0
- removed link cylindrical_1_0
- removed link cylindrical_1_3
- removed link cylindrical_1_6
- removed link cylindrical_1_9
- removed link cylindrical_2_0
- removed link cylindrical_2_3
- removed link cylindrical_4_0
- removed link cylindrical_6_0
- removed link cylindrical_7_0
- removed link cylindrical_9_0
- removed link gear_housing
- removed link gpa72mr2060_a_pud_b
- removed link gpa72mr2060_a_pud_b_1
- removed link gpa72mr2060_a_puef_b
- removed link hand_motor
- removed link hex_socket_head_cap_screw_m1_6x0_35_x_12
- removed link hex_socket_head_cap_screw_m1_6x0_35_x_12_1
- removed link l_shape_1
- removed link m4x20
- removed link m4x20_1
- removed link m4x20_2
- removed link m4x20_3
- removed link mgl17_g10__1_
- removed link mgl17_g10__2_
- removed link motor
- removed link motor_1
- removed link motor_2
- removed link netrf12_25
- removed link netrf12_25_1
- removed link netrf12_25_2
- removed link netrf12_25_3
- removed link netrf12_25_4
- removed link netrf12_60
- removed link netrf12_60_1
- removed link netrf12_60_2
- removed link netrf12_60_3
- removed link netrf12_60_4
- removed link netrf12_60_5
- removed link netrf12_60_6
- removed link parallel_1_0
- removed link parallel_1_1
- removed link parallel_1_2
- removed link parallel_3_0
- removed link parallel_3_1
- removed link parallel_3_2
- removed link part_1
- removed link part_12
- removed link part_13
- removed link part_13_1
- removed link part_13_2
- removed link part_14
- removed link part_14_1
- removed link part_15
- removed link part_15_1
- removed link part_16
- removed link part_16_1
- removed link part_1_1
- removed link part_1_10
- removed link part_1_100
- removed link part_1_101
- removed link part_1_102
- removed link part_1_103
- removed link part_1_104
- removed link part_1_105
- removed link part_1_106
- removed link part_1_107
- removed link part_1_108
- removed link part_1_109
- removed link part_1_11
- removed link part_1_110
- removed link part_1_111
- removed link part_1_112
- removed link part_1_113
- removed link part_1_114
- removed link part_1_115
- removed link part_1_116
- removed link part_1_117
- removed link part_1_118
- removed link part_1_119
- removed link part_1_12
- removed link part_1_120
- removed link part_1_121
- removed link part_1_122
- removed link part_1_123
- removed link part_1_124
- removed link part_1_125
- removed link part_1_126
- removed link part_1_127
- removed link part_1_128
- removed link part_1_129
- removed link part_1_13
- removed link part_1_130
- removed link part_1_131
- removed link part_1_132
- removed link part_1_133
- removed link part_1_134
- removed link part_1_135
- removed link part_1_136
- removed link part_1_137
- removed link part_1_138
- removed link part_1_139
- removed link part_1_14
- removed link part_1_140
- removed link part_1_141
- removed link part_1_142
- removed link part_1_143
- removed link part_1_144
- removed link part_1_145
- removed link part_1_146
- removed link part_1_147
- removed link part_1_148
- removed link part_1_149
- removed link part_1_15
- removed link part_1_150
- removed link part_1_151
- removed link part_1_152
- removed link part_1_153
- removed link part_1_154
- removed link part_1_155
- removed link part_1_156
- removed link part_1_157
- removed link part_1_158
- removed link part_1_159
- removed link part_1_16
- removed link part_1_160
- removed link part_1_161
- removed link part_1_162
- removed link part_1_163
- removed link part_1_164
- removed link part_1_165
- removed link part_1_166
- removed link part_1_167
- removed link part_1_168
- removed link part_1_169
- removed link part_1_17
- removed link part_1_170
- removed link part_1_171
- removed link part_1_172
- removed link part_1_173
- removed link part_1_174
- removed link part_1_175
- removed link part_1_176
- removed link part_1_177
- removed link part_1_178
- removed link part_1_179
- removed link part_1_18
- removed link part_1_180
- removed link part_1_181
- removed link part_1_182
- removed link part_1_183
- removed link part_1_184
- removed link part_1_185
- removed link part_1_186
- removed link part_1_187
- removed link part_1_2
- removed link part_1_22
- removed link part_1_23
- removed link part_1_27
- removed link part_1_28
- removed link part_1_29
- removed link part_1_3
- removed link part_1_31
- removed link part_1_32
- removed link part_1_34
- removed link part_1_36
- removed link part_1_37
- removed link part_1_38
- removed link part_1_39
- removed link part_1_4
- removed link part_1_40
- removed link part_1_41
- removed link part_1_42
- removed link part_1_43
- removed link part_1_44
- removed link part_1_45
- removed link part_1_47
- removed link part_1_49
- removed link part_1_5
- removed link part_1_50
- removed link part_1_51
- removed link part_1_52
- removed link part_1_53
- removed link part_1_54
- removed link part_1_55
- removed link part_1_56
- removed link part_1_57
- removed link part_1_58
- removed link part_1_59
- removed link part_1_6
- removed link part_1_60
- removed link part_1_61
- removed link part_1_62
- removed link part_1_63
- removed link part_1_64
- removed link part_1_65
- removed link part_1_66
- removed link part_1_67
- removed link part_1_68
- removed link part_1_69
- removed link part_1_7
- removed link part_1_70
- removed link part_1_71
- removed link part_1_72
- removed link part_1_73
- removed link part_1_74
- removed link part_1_75
- removed link part_1_76
- removed link part_1_77
- removed link part_1_78
- removed link part_1_79
- removed link part_1_8
- removed link part_1_80
- removed link part_1_81
- removed link part_1_82
- removed link part_1_83
- removed link part_1_84
- removed link part_1_85
- removed link part_1_86
- removed link part_1_87
- removed link part_1_88
- removed link part_1_89
- removed link part_1_9
- removed link part_1_90
- removed link part_1_91
- removed link part_1_92
- removed link part_1_93
- removed link part_1_94
- removed link part_1_95
- removed link part_1_96
- removed link part_1_97
- removed link part_1_98
- removed link part_1_99
- removed link part_2
- removed link part_2_1
- removed link part_2_2
- removed link planar_1_0
- removed link planar_1_1
- removed link planar_1_10
- removed link planar_1_11
- removed link planar_1_15
- removed link planar_1_16
- removed link planar_1_5
- removed link planar_1_6
- removed link planar_2_0
- removed link planar_2_1
- removed link planar_2_5
- removed link planar_2_6
- removed link planar_3_0
- removed link planar_3_1
- removed link planar_3_10
- removed link planar_3_11
- removed link planar_3_5
- removed link planar_3_6
- removed link planar_4_0
- removed link planar_4_1
- removed link planar_5_0
- removed link planar_5_1
- removed link planar_5_5
- removed link planar_5_6
- removed link planar_6_0
- removed link planar_6_1
- removed link planar_7_0
- removed link planar_7_1
- removed link planar_8_0
- removed link planar_8_1
- removed link rev_11_3174_p01_customer_blank_1
- removed link rev_11_3174_p02_customer_blank
- removed link rev_11_3174_p02_customer_blank_1
- removed link robaj10_ba
- removed link robaj10_bl
- removed link root
- removed link set_screw_8_32_0_328
- removed link shaft
- removed link shoulder_to_elbow_belt
- removed link skeleton_enclousre
- removed link spur_assembly__1_
- removed link spur_gear__12_teeth_
- removed link spur_gear__36_teeth_
- removed link ss__1__1
- removed link ss_arm_ss
- removed link ss_arm_ss_1
- removed link ss_base_ss
- removed link ss_base_ss_1
- removed link stand_off
- removed link stand_off_1
- removed link stwn8
- removed link stwn8_1
- removed link stwn8_2
- removed link stwn8_3
- removed link stwn8_4
- removed link stwn8_5
- removed link sw输入端盖
- removed link sw输入端盖_1
- removed link uxcell_51101_thrust_ball_bearings
- removed link wrist_differential_stepped_shaft
- removed link 输出轴
- removed link 输出轴_1
- added link Elbowgroup
- added link base_center
- added link truss_group
- added link world
- link base_plate_wall_left: geometry collision mesh filename=package://arm_assembly/meshes/Base Plate Wall Left.stl scale=1 1 1; visual mesh filename=package://arm_assembly/meshes/Base Plate Wall Left.stl scale=1 1 1
- link base_plate_wall_right: geometry collision mesh filename=package://arm_assembly/meshes/Base Plate Wall Right.stl scale=1 1 1; visual mesh filename=package://arm_assembly/meshes/Base Plate Wall Right.stl scale=1 1 1
- link left_elbow_truss: geometry collision mesh filename=package://arm_assembly/meshes/Left Elbow Truss.stl scale=1 1 1; visual mesh filename=package://arm_assembly/meshes/Left Elbow Truss.stl scale=1 1 1
- link right_elbow_truss: geometry collision mesh filename=package://arm_assembly/meshes/Right Elbow Truss.stl scale=1 1 1; visual mesh filename=package://arm_assembly/meshes/Right Elbow Truss.stl scale=1 1 1
- link truss_left: mass 0.355071 -> 0.379638; geometry collision mesh filename=package://arm_assembly/meshes/Truss Left.stl scale=1 1 1; visual mesh filename=package://arm_assembly/meshes/Truss Left.stl scale=1 1 1
- link truss_right: mass 0.379638 -> 0.355071; geometry collision mesh filename=package://arm_assembly/meshes/Truss Right.stl scale=1 1 1; visual mesh filename=package://arm_assembly/meshes/Truss Right.stl scale=1 1 1
Joints:
- removed joint cylindrical_10_1
- removed joint cylindrical_10_2
- removed joint cylindrical_12_1
- removed joint cylindrical_12_2
- removed joint cylindrical_1_1
- removed joint cylindrical_1_10
- removed joint cylindrical_1_11
- removed joint cylindrical_1_2
- removed joint cylindrical_1_4
- removed joint cylindrical_1_5
- removed joint cylindrical_1_7
- removed joint cylindrical_1_8
- removed joint cylindrical_2_1
- removed joint cylindrical_2_2
- removed joint cylindrical_2_4
- removed joint cylindrical_2_5
- removed joint cylindrical_4_1
- removed joint cylindrical_4_2
- removed joint cylindrical_6_1
- removed joint cylindrical_6_2
- removed joint cylindrical_7_1
- removed joint cylindrical_7_2
- removed joint cylindrical_9_1
- removed joint cylindrical_9_2
- removed joint dof_3_0
- removed joint fastened_100_0
- removed joint fastened_101_0
- removed joint fastened_102_0
- removed joint fastened_103_0
- removed joint fastened_104_0
- removed joint fastened_105_0
- removed joint fastened_106_0
- removed joint fastened_107_0
- removed joint fastened_108_0
- removed joint fastened_109_0
- removed joint fastened_10_0
- removed joint fastened_10_1
- removed joint fastened_110_0
- removed joint fastened_111_0
- removed joint fastened_112_0
- removed joint fastened_113_0
- removed joint fastened_114_0
- removed joint fastened_115_0
- removed joint fastened_116_0
- removed joint fastened_117_0
- removed joint fastened_118_0
- removed joint fastened_119_0
- removed joint fastened_11_0
- removed joint fastened_11_1
- removed joint fastened_11_2
- removed joint fastened_120_0
- removed joint fastened_121_0
- removed joint fastened_122_0
- removed joint fastened_123_0
- removed joint fastened_124_0
- removed joint fastened_125_0
- removed joint fastened_126_0
- removed joint fastened_127_0
- removed joint fastened_128_0
- removed joint fastened_129_0
- removed joint fastened_12_0
- removed joint fastened_12_1
- removed joint fastened_12_2
- removed joint fastened_12_3
- removed joint fastened_130_0
- removed joint fastened_131_0
- removed joint fastened_132_0
- removed joint fastened_133_0
- removed joint fastened_134_0
- removed joint fastened_135_0
- removed joint fastened_136_0
- removed joint fastened_137_0
- removed joint fastened_138_0
- removed joint fastened_139_0
- removed joint fastened_13_0
- removed joint fastened_13_1
- removed joint fastened_13_2
- removed joint fastened_140_0
- removed joint fastened_141_0
- removed joint fastened_14_0
- removed joint fastened_14_1
- removed joint fastened_14_2
- removed joint fastened_15_0
- removed joint fastened_15_1
- removed joint fastened_15_2
- removed joint fastened_16_0
- removed joint fastened_16_1
- removed joint fastened_16_2
- removed joint fastened_17_0
- removed joint fastened_17_1
- removed joint fastened_17_2
- removed joint fastened_18_0
- removed joint fastened_18_1
- removed joint fastened_18_2
- removed joint fastened_19_0
- removed joint fastened_19_1
- removed joint fastened_1_0
- removed joint fastened_1_1
- removed joint fastened_1_2
- removed joint fastened_20_0
- removed joint fastened_20_1
- removed joint fastened_21_0
- removed joint fastened_21_1
- removed joint fastened_22_0
- removed joint fastened_23_0
- removed joint fastened_23_1
- removed joint fastened_23_2
- removed joint fastened_24_0
- removed joint fastened_24_1
- removed joint fastened_25_0
- removed joint fastened_25_1
- removed joint fastened_26_0
- removed joint fastened_26_1
- removed joint fastened_27_0
- removed joint fastened_27_1
- removed joint fastened_28_0
- removed joint fastened_28_1
- removed joint fastened_29_0
- removed joint fastened_29_1
- removed joint fastened_2_0
- removed joint fastened_2_1
- removed joint fastened_2_2
- removed joint fastened_2_3
- removed joint fastened_30_0
- removed joint fastened_30_1
- removed joint fastened_31_0
- removed joint fastened_31_1
- removed joint fastened_31_2
- removed joint fastened_32_0
- removed joint fastened_33_0
- removed joint fastened_34_0
- removed joint fastened_35_0
- removed joint fastened_36_0
- removed joint fastened_37_0
- removed joint fastened_38_0
- removed joint fastened_39_0
- removed joint fastened_3_0
- removed joint fastened_3_1
- removed joint fastened_3_2
- removed joint fastened_3_3
- removed joint fastened_3_4
- removed joint fastened_40_0
- removed joint fastened_41_0
- removed joint fastened_42_0
- removed joint fastened_43_0
- removed joint fastened_44_0
- removed joint fastened_45_0
- removed joint fastened_46_0
- removed joint fastened_47_0
- removed joint fastened_48_0
- removed joint fastened_49_0
- removed joint fastened_4_0
- removed joint fastened_4_1
- removed joint fastened_4_2
- removed joint fastened_50_0
- removed joint fastened_51_0
- removed joint fastened_54_0
- removed joint fastened_55_0
- removed joint fastened_56_0
- removed joint fastened_57_0
- removed joint fastened_58_0
- removed joint fastened_59_0
- removed joint fastened_5_0
- removed joint fastened_5_1
- removed joint fastened_5_2
- removed joint fastened_60_0
- removed joint fastened_61_0
- removed joint fastened_62_0
- removed joint fastened_63_0
- removed joint fastened_64_0
- removed joint fastened_65_0
- removed joint fastened_66_0
- removed joint fastened_67_0
- removed joint fastened_68_0
- removed joint fastened_69_0
- removed joint fastened_6_0
- removed joint fastened_6_1
- removed joint fastened_6_2
- removed joint fastened_6_3
- removed joint fastened_6_4
- removed joint fastened_70_0
- removed joint fastened_71_0
- removed joint fastened_72_0
- removed joint fastened_73_0
- removed joint fastened_74_0
- removed joint fastened_75_0
- removed joint fastened_76_0
- removed joint fastened_77_0
- removed joint fastened_78_0
- removed joint fastened_79_0
- removed joint fastened_7_0
- removed joint fastened_7_1
- removed joint fastened_7_2
- removed joint fastened_7_3
- removed joint fastened_7_4
- removed joint fastened_80_0
- removed joint fastened_81_0
- removed joint fastened_82_0
- removed joint fastened_83_0
- removed joint fastened_84_0
- removed joint fastened_85_0
- removed joint fastened_86_0
- removed joint fastened_87_0
- removed joint fastened_88_0
- removed joint fastened_89_0
- removed joint fastened_8_0
- removed joint fastened_8_1
- removed joint fastened_8_2
- removed joint fastened_8_3
- removed joint fastened_90_0
- removed joint fastened_91_0
- removed joint fastened_92_0
- removed joint fastened_93_0
- removed joint fastened_94_0
- removed joint fastened_95_0
- removed joint fastened_96_0
- removed joint fastened_97_0
- removed joint fastened_98_0
- removed joint fastened_99_0
- removed joint fastened_9_0
- removed joint fastened_9_1
- removed joint fastened_9_2
- removed joint fastened_9_3
- removed joint group_1_fastened_joint_0
- removed joint group_1_fastened_joint_1
- removed joint group_2_fastened_joint_0
- removed joint group_2_fastened_joint_1
- removed joint group_2_fastened_joint_2
- removed joint group_2_fastened_joint_3
- removed joint group_2_fastened_joint_4
- removed joint group_2_fastened_joint_5
- removed joint group_2_fastened_joint_6
- removed joint group_3_fastened_joint_0
- removed joint group_3_fastened_joint_1
- removed joint group_3_fastened_joint_10
- removed joint group_3_fastened_joint_11
- removed joint group_3_fastened_joint_12
- removed joint group_3_fastened_joint_13
- removed joint group_3_fastened_joint_14
- removed joint group_3_fastened_joint_15
- removed joint group_3_fastened_joint_16
- removed joint group_3_fastened_joint_17
- removed joint group_3_fastened_joint_2
- removed joint group_3_fastened_joint_3
- removed joint group_3_fastened_joint_4
- removed joint group_3_fastened_joint_5
- removed joint group_3_fastened_joint_6
- removed joint group_3_fastened_joint_7
- removed joint group_3_fastened_joint_8
- removed joint group_3_fastened_joint_9
- removed joint group_5_fastened_joint_0
- removed joint group_5_fastened_joint_1
- removed joint group_6_fastened_joint_0
- removed joint group_6_fastened_joint_1
- removed joint group_6_fastened_joint_2
- removed joint group_6_fastened_joint_3
- removed joint group_6_fastened_joint_4
- removed joint group_7_fastened_joint_0
- removed joint group_8_fastened_joint_0
- removed joint group_8_fastened_joint_1
- removed joint group_8_fastened_joint_2
- removed joint group_9_fastened_joint_0
- removed joint group_9_fastened_joint_1
- removed joint hanging_node_to_root_joint_0
- removed joint hanging_node_to_root_joint_1
- removed joint parallel_1_3
- removed joint parallel_1_4
- removed joint parallel_1_5
- removed joint parallel_1_6
- removed joint parallel_3_3
- removed joint parallel_3_4
- removed joint parallel_3_5
- removed joint parallel_3_6
- removed joint planar_1_12
- removed joint planar_1_13
- removed joint planar_1_14
- removed joint planar_1_17
- removed joint planar_1_18
- removed joint planar_1_19
- removed joint planar_1_2
- removed joint planar_1_3
- removed joint planar_1_4
- removed joint planar_1_7
- removed joint planar_1_8
- removed joint planar_1_9
- removed joint planar_2_2
- removed joint planar_2_3
- removed joint planar_2_4
- removed joint planar_2_7
- removed joint planar_2_8
- removed joint planar_2_9
- removed joint planar_3_12
- removed joint planar_3_13
- removed joint planar_3_14
- removed joint planar_3_2
- removed joint planar_3_3
- removed joint planar_3_4
- removed joint planar_3_7
- removed joint planar_3_8
- removed joint planar_3_9
- removed joint planar_4_2
- removed joint planar_4_3
- removed joint planar_4_4
- removed joint planar_5_2
- removed joint planar_5_3
- removed joint planar_5_4
- removed joint planar_5_7
- removed joint planar_5_8
- removed joint planar_5_9
- removed joint planar_6_2
- removed joint planar_6_3
- removed joint planar_6_4
- removed joint planar_7_2
- removed joint planar_7_3
- removed joint planar_7_4
- removed joint planar_8_2
- removed joint planar_8_3
- removed joint planar_8_4
- removed joint revolute_10_0
- removed joint revolute_10_1
- removed joint revolute_11_0
- removed joint revolute_1_0
- removed joint revolute_1_1
- removed joint revolute_1_2
- removed joint revolute_1_3
- removed joint revolute_2_0
- removed joint revolute_2_1
- removed joint revolute_3_0
- removed joint revolute_3_1
- removed joint revolute_3_2
- removed joint revolute_3_3
- removed joint revolute_4_0
- removed joint revolute_4_1
- removed joint revolute_4_2
- removed joint revolute_4_3
- removed joint revolute_5_0
- removed joint revolute_5_1
- removed joint revolute_6_0
- removed joint revolute_6_1
- removed joint revolute_6_2
- removed joint revolute_7_0
- removed joint revolute_8_0
- removed joint slider_1_0
- removed joint slider_2_0
- removed joint temporary_group_fastened_joint_0
- removed joint temporary_group_fastened_joint_1
- removed joint temporary_group_fastened_joint_2
- removed joint temporary_group_fastened_joint_3
- removed joint temporary_group_fastened_joint_4
- removed joint temporary_group_fastened_joint_5
- removed joint temporary_group_fastened_joint_6
- removed joint temporary_group_fastened_joint_7
- added joint base_left_joint: type fixed, parent base_center, child base_plate_wall_left, origin xyz=0 0.1 0 rpy=0 0 0
- added joint base_right_joint: type fixed, parent base_center, child base_plate_wall_right, origin xyz=0 -0.1 0 rpy=0 0 3.14159
- added joint base_rotation: type revolute, parent world, child base_center, origin xyz=0 0 0 rpy=0 0 0, axis 0 0 1, limit lower=-3.14159 upper=3.14159 effort=50 velocity=2
- added joint left_elbow: type fixed, parent Elbowgroup, child left_elbow_truss, origin xyz=0.15 0.025 0 rpy=3.14159 0 1.5708 
- added joint left_truss_joint: type fixed, parent truss_group, child truss_left, origin xyz=0.23 0 -0.07 rpy=0 0 0
- added joint right_elbow: type fixed, parent Elbowgroup, child right_elbow_truss, origin xyz=0.285 -0.078 -0.01 rpy=3.14159 0 1.5708 
- added joint right_truss_joint: type fixed, parent truss_group, child truss_right, origin xyz=0.23 0 0.07 rpy=0 0 0
- added joint truss_main_elbow: type revolute, parent truss_group, child Elbowgroup, origin xyz=0.23 0 0.03 rpy=1.5708 0 0, axis 0 1 0, limit lower=-3.14 upper=3.14 effort=50 velocity=2
- added joint truss_main_joint: type revolute, parent base_center, child truss_group, origin xyz=0.065 0 0.03 rpy=1.5708 0 0, axis 0 0 1, limit lower=-1.57 upper=3.14 effort=50 velocity=2
