Commit message: FIXED URDF SIMPLIFIED

File: arm_assembly/src/description/arm_assembly_simplified.urdf (robot description, URDF)
Before this commit: robot simple_arm, 10 links, 9 joints
Links:
- link left_elbow_truss: geometry collision mesh filename=package://arm_assembly/meshes/Left Elbow Truss.stl scale=1 1 1; visual mesh filename=package://arm_assembly/meshes/Left Elbow Truss.stl scale=1 1 1
- link right_elbow_truss: geometry collision mesh filename=package://arm_assembly/meshes/Right Elbow Truss.stl scale=1 1 1; visual mesh filename=package://arm_assembly/meshes/Right Elbow Truss.stl scale=1 1 1
- link truss_left: mass 0.355071 -> 0.379638; geometry collision mesh filename=package://arm_assembly/meshes/Truss Left.stl scale=1 1 1; visual mesh filename=package://arm_assembly/meshes/Truss Left.stl scale=1 1 1
- link truss_right: mass 0.379638 -> 0.355071; geometry collision mesh filename=package://arm_assembly/meshes/Truss Right.stl scale=1 1 1; visual mesh filename=package://arm_assembly/meshes/Truss Right.stl scale=1 1 1
Joints:
- joint left_elbow: origin xyz=0.15 0.045 0 rpy=3.14159 0 1.5708  -> xyz=0.15 0.025 0 rpy=3.14159 0 1.5708 
- joint left_truss_joint: origin xyz=0 0 -0.1 rpy=0 0 0 -> xyz=0.23 0 -0.07 rpy=0 0 0
- joint right_elbow: origin xyz=0.285 -0.11 -0.01 rpy=3.14159 0 1.5708  -> xyz=0.285 -0.078 -0.01 rpy=3.14159 0 1.5708 
- joint right_truss_joint: origin xyz=0 0 0.085 rpy=0 0 0 -> xyz=0.23 0 0.07 rpy=0 0 0
